Commit message: added mapping.launch

File: my_robot/urdf/my_robot.xacro (robot description, xacro)
@@ -150,4 +150,11 @@
     <axis xyz="0 1 0" rpy="0 0 0"/>
   </joint>
+  <joint name="camera_optical_joint" type="fixed">
+    <origin xyz="0.2 0 0" rpy="0 0 0"/>
+    <parent link="chassis"/>
+    <child link="camera_link_optical"/>
+  </joint>
+  <link name="camera_link_optical">
+  </link>
   <link name='hokuyo'>
     <pose>0 0 0 0 0 0</pose>
@@ -170,5 +177,4 @@
       <origin xyz="0 0 0" rpy="0 1.5707 0"/>
       <geometry>
-        <!--box size=".1 .1 .1"/-->
         <mesh filename="package://my_robot/meshes/hokuyo.dae"/>
       </geometry>

Commit message: fixed typos in the urdf files

File: my_robot/urdf/my_robot.xacro (robot description, xacro)
@@ -150,11 +150,11 @@
     <axis xyz="0 1 0" rpy="0 0 0"/>
   </joint>
-  <joint name="camera_optical_joint" type="fixed">
+  <link name="camera_RGBD">
+  </link>
+  <joint name="camera_joint_RGBD" type="fixed">
     <origin xyz="0.2 0 0" rpy="0 0 0"/>
     <parent link="chassis"/>
-    <child link="camera_link_optical"/>
-  </joint>
-  <link name="camera_link_optical">
-  </link>
+    <child link="camera_RGBD"/>
+  </joint>
   <link name='hokuyo'>
     <pose>0 0 0 0 0 0</pose>
